File: kicad/IS31FL3736_Dev.sch (KiCad schematic (older format))
At the start: 57 parts, among them J1 Daisy IN, J2 Daisy OUT, U1 IS31FL3736

Commit message: Layout done
Parts:
- removed C2, C3, C4: 0.47μF, Capacitor_SMD:C_0805_2012Metric, symbol Device:C
- removed J2: Daisy OUT, Connector_PinHeader_2.54mm:PinHeader_1x09_P2.54mm_Horizontal, symbol Connector:Conn_01x09_Female
- added J2: Bottom_SW_Connector, Pin_Headers:Pin_Header_Straight_1x12_Pitch2.54mm, symbol Connector:Conn_01x12_Female
- added J3: Top_SW_Connector, Pin_Headers:Pin_Header_Straight_1x12_Pitch2.54mm, symbol Connector:Conn_01x12_Male
- added J4: Bottom_CS_Connector, Pin_Headers:Pin_Header_Straight_1x08_Pitch2.54mm, symbol Connector:Conn_01x08_Female
- added J5: Top_CS_Connector, Pin_Headers:Pin_Header_Straight_1x08_Pitch2.54mm, symbol Connector:Conn_01x08_Male
- D1, D10, D11, D12, D13, D14, D15, D16, D17, D18, D19, D2, D20, D21, D22, D23, D24, D25, D26, D27, D28, D29, D3, D30, D31, D32, D4, D5, D6, D7, D8, D9: MPN (none) -> AAA3528LSEEZGKQBKS
- JP1, JP2, JP3, JP4, JP5, JP6, JP8: footprint Jumper:SolderJumper-2_P1.3mm_Open_Pad1.0x1.5mm -> Jumper:SolderJumper-2_P1.3mm_Open_RoundedPad1.0x1.5mm
- JP7: value SLC ADDR2 -> SCL ADDR2; footprint Jumper:SolderJumper-2_P1.3mm_Open_Pad1.0x1.5mm -> Jumper:SolderJumper-2_P1.3mm_Open_RoundedPad1.0x1.5mm
- R1, R2, R3, R4, R5: footprint Resistor_SMD:R_0805_2012Metric -> Resistors_SMD:R_0805
- R6: footprint Resistor_SMD:R_2512_6332Metric -> Resistors_SMD:R_0805
- U1: footprint Package_DFN_QFN:QFN-40-1EP_5x5mm_P0.4mm_EP3.8x3.8mm -> Housings_DFN_QFN:QFN-40-1EP_5x5mm_Pitch0.4mm; MPN (none) -> IS31FL3736
Connections:
- net labels added: BCS1, BCS2, BCS3, BCS4, BCS5, BCS6, BCS7, BCS8, BSW1, BSW10, BSW11, BSW12, BSW2, BSW3, BSW4, BSW5, BSW6, BSW7, BSW8, BSW9, TCS1, TCS2, TCS3, TCS4, TCS5, TCS6, TCS7, TCS8, TSW1, TSW10, TSW11, TSW12, TSW2, TSW3, TSW4, TSW5, TSW6, TSW7, TSW8, TSW9
- net labels removed: CS1, CS2, CS3, CS4, CS5, CS6, CS7, CS8, SW1, SW10, SW11, SW12, SW2, SW3, SW4, SW5, SW6, SW7, SW8, SW9
- wire segments 303 -> 333
Other:
- note added: "Optional"
- note added: "SBD - Pulled low to disable the chip\nThe MCU will need to pull this high."
- moved on the sheet: C5, C6, C7, J1

Commit message: Update to SBD pullup
Parts:
- J1: value Daisy IN -> I/O Connector
Connections:
- net GND: no longer R4.1
- net Vio: now also R4.2
- net ~SDB: now also R4.1; no longer R4.2
Other:
- moved on the sheet: JP1, JP2, JP3, JP4, JP5, JP6, JP7, JP8, R1, R2, R3, R4
