File: kicad/IS31FL3736_Dev.sch (KiCad schematic (older format))
At the start: 57 parts, among them J1 I/O Connector, J2 Bottom_SW_Connector, J3 Top_SW_Connector, J4 Bottom_CS_Connector, J5 Top_CS_Connector, U1 IS31FL3736

Commit message: Archived for KiCad 5.0.1
Parts:
- D1, D10, D11, D12, D13, D14, D15, D16, D17, D18, D19, D2, D20, D21, D22, D23, D24, D25, D26, D27, D28, D29, D3, D30, D31, D32, D4, D5, D6, D7, D8, D9: symbol Device:LED_RGBA -> IS31FL3736_Dev-rescue:LED_RGBA-Device
- U1: symbol Driver_LED:IS31FL3736 -> IS31FL3736_Dev-rescue:IS31FL3736-Driver_LED
Changed lines of the file:
@@
 EESchema Schematic File Version 4
-EELAYER 30 0
+LIBS:IS31FL3736_Dev-cache
+EELAYER 26 0
 EELAYER END
 $Descr A3 16535 11693
@@
 PVCC_17
 $Comp
-L Driver_LED:IS31FL3736 U1
+L IS31FL3736_Dev-rescue:IS31FL3736-Driver_LED U1
 U 1 1 5E0A16A5
 P 4450 5350
@@
 $EndComp
 $Comp
-L Device:LED_RGBA D5
+L IS31FL3736_Dev-rescue:LED_RGBA-Device D5
 U 1 1 5E0C1EB9
 P 8250 6100
@@
 $EndComp
 $Comp
-L Device:LED_RGBA D6
+L IS31FL3736_Dev-rescue:LED_RGBA-Device D6
 U 1 1 5E0C1EC3
 P 8250 6950
@@
 $EndComp
 $Comp
-L Device:LED_RGBA D7
+L IS31FL3736_Dev-rescue:LED_RGBA-Device D7
 U 1 1 5E0C1ECD
 P 8250 7850
@@
 $EndComp
 $Comp
-L Device:LED_RGBA D8
+L IS31FL3736_Dev-rescue:LED_RGBA-Device D8
 U 1 1 5E0C1ED7
 P 8250 8700
@@
 $EndComp
 $Comp
-L Device:LED_RGBA D9
+L IS31FL3736_Dev-rescue:LED_RGBA-Device D9
 U 1 1 5E27EDE8
 P 9450 6100
@@
 $EndComp
 $Comp
-L Device:LED_RGBA D10
+L IS31FL3736_Dev-rescue:LED_RGBA-Device D10
 U 1 1 5E27EDF2
 P 9450 6950
@@
 $EndComp
 $Comp
-L Device:LED_RGBA D11
+L IS31FL3736_Dev-rescue:LED_RGBA-Device D11
 U 1 1 5E27EDFC
 P 9450 7850
@@
 $EndComp
 $Comp
-L Device:LED_RGBA D12
+L IS31FL3736_Dev-rescue:LED_RGBA-Device D12
 U 1 1 5E27EE06
 P 9450 8700
@@
 $EndComp
 $Comp
-L Device:LED_RGBA D13
+L IS31FL3736_Dev-rescue:LED_RGBA-Device D13
 U 1 1 5E27EE10
 P 10500 6100
@@
 $EndComp
 $Comp
-L Device:LED_RGBA D14
+L IS31FL3736_Dev-rescue:LED_RGBA-Device D14
 U 1 1 5E27EE1A
 P 10500 6950
@@
 $EndComp
 $Comp
-L Device:LED_RGBA D15
+L IS31FL3736_Dev-rescue:LED_RGBA-Device D15
 U 1 1 5E27EE24
 P 10500 7850
@@
 $EndComp
 $Comp
-L Device:LED_RGBA D16
+L IS31FL3736_Dev-rescue:LED_RGBA-Device D16
 U 1 1 5E27EE2E
 P 10500 8700
@@
 $EndComp
 $Comp
-L Device:LED_RGBA D17
+L IS31FL3736_Dev-rescue:LED_RGBA-Device D17
 U 1 1 5E2B81E8
 P 11650 6100
@@
 $EndComp
 $Comp
-L Device:LED_RGBA D18
+L IS31FL3736_Dev-rescue:LED_RGBA-Device D18
 U 1 1 5E2B81F2
 P 11650 6950
@@
 $EndComp
 $Comp
-L Device:LED_RGBA D19
+L IS31FL3736_Dev-rescue:LED_RGBA-Device D19
 U 1 1 5E2B81FC
 P 11650 7850
@@
 $EndComp
 $Comp
-L Device:LED_RGBA D20
+L IS31FL3736_Dev-rescue:LED_RGBA-Device D20
 U 1 1 5E2B8206
 P 11650 8700
@@
 $EndComp
 $Comp
-L Device:LED_RGBA D21
+L IS31FL3736_Dev-rescue:LED_RGBA-Device D21
 U 1 1 5E2B8210
 P 12700 6100
@@
 $EndComp
 $Comp
-L Device:LED_RGBA D22
+L IS31FL3736_Dev-rescue:LED_RGBA-Device D22
 U 1 1 5E2B821A
 P 12700 6950
@@
 $EndComp
 $Comp
-L Device:LED_RGBA D23
+L IS31FL3736_Dev-rescue:LED_RGBA-Device D23
 U 1 1 5E2B8224
 P 12700 7850
@@
 $EndComp
 $Comp
-L Device:LED_RGBA D24
+L IS31FL3736_Dev-rescue:LED_RGBA-Device D24
 U 1 1 5E2B822E
 P 12700 8700
@@
 $EndComp
 $Comp
-L Device:LED_RGBA D25
+L IS31FL3736_Dev-rescue:LED_RGBA-Device D25
 U 1 1 5E2B8282
 P 13900 6100
@@
 $EndComp
 $Comp
-L Device:LED_RGBA D26
+L IS31FL3736_Dev-rescue:LED_RGBA-Device D26
 U 1 1 5E2B828C
 P 13900 6950
@@
 $EndComp
 $Comp
-L Device:LED_RGBA D27
+L IS31FL3736_Dev-rescue:LED_RGBA-Device D27
 U 1 1 5E2B8296
 P 13900 7850
@@
 $EndComp
 $Comp
-L Device:LED_RGBA D28
+L IS31FL3736_Dev-rescue:LED_RGBA-Device D28
 U 1 1 5E2B82A0
 P 13900 8700
@@
 $EndComp
 $Comp
-L Device:LED_RGBA D29
+L IS31FL3736_Dev-rescue:LED_RGBA-Device D29
 U 1 1 5E2B82AA
 P 14950 6100
@@
 $EndComp
 $Comp
-L Device:LED_RGBA D30
+L IS31FL3736_Dev-rescue:LED_RGBA-Device D30
 U 1 1 5E2B82B4
 P 14950 6950
@@
 $EndComp
 $Comp
-L Device:LED_RGBA D31
+L IS31FL3736_Dev-rescue:LED_RGBA-Device D31
 U 1 1 5E2B82BE
 P 14950 7850
@@
 $EndComp
 $Comp
-L Device:LED_RGBA D32
+L IS31FL3736_Dev-rescue:LED_RGBA-Device D32
 U 1 1 5E2B82C8
 P 14950 8700
@@
 IICRST
 $Comp
-L Device:LED_RGBA D4
+L IS31FL3736_Dev-rescue:LED_RGBA-Device D4
 U 1 1 5E0AF8D7
 P 7200 8700
@@
 $EndComp
 $Comp
-L Device:LED_RGBA D3
+L IS31FL3736_Dev-rescue:LED_RGBA-Device D3
 U 1 1 5E0AF8CD
 P 7200 7850
@@
 $EndComp
 $Comp
-L Device:LED_RGBA D2
+L IS31FL3736_Dev-rescue:LED_RGBA-Device D2
 U 1 1 5E0A8588
 P 7200 6950
@@
 $EndComp
 $Comp
-L Device:LED_RGBA D1
+L IS31FL3736_Dev-rescue:LED_RGBA-Device D1
 U 1 1 5E0A59CC
 P 7200 6100
